Commit message: feat: Phase 2 complete — full 6DOF URDF with STL meshes and joint control
- arm.urdf.xacro: all 6 revolute joints + fixed tool_link
- Joint axes: J1 Z, J2 Y, J3 Y, J4 X, J5 Y, J6 Z
- STL meshes exported from Onshape arm_6dof_ros2 document
- Joint limits set, inertial properties defined for all links
- RViz config updated with full arm display

File: 01_6dof_arm/arm_description/urdf/arm.urdf.xacro (robot description, xacro)
@@ -2,40 +2,216 @@
 <robot xmlns:xacro="http://www.ros.org/wiki/xacro" name="arm_6dof">
   <!-- ============================================================
-       arm.urdf.xacro
-       6DOF robotic arm - base link only (Phase 1 stub)
-       We will add joints and links one by one in Phase 2
+       arm.urdf.xacro — Full 6DOF arm
+       All dimensions in metres. Joints stack vertically along Z.
+       Link lengths:
+         base   : 40mm
+         link_1 : 80mm
+         link_2 : 120mm
+         link_3 : 100mm
+         link_4 : 40mm
+         link_5 : 35mm
+         link_6 : 15mm
        ============================================================ -->
-  <!-- PROPERTY: change dimensions in one place, reflects everywhere -->
-  <xacro:property name="base_radius" value="0.05"/>
-  <xacro:property name="base_height" value="0.04"/>
-  <xacro:property name="base_mass"   value="1.0"/>
-  <!-- BASE LINK: fixed mounting point of the arm -->
+  <!-- ===================== MATERIALS ===================== -->
+  <material name="dark_grey">
+    <color rgba="0.2 0.2 0.2 1.0"/>
+  </material>
+  <material name="light_grey">
+    <color rgba="0.7 0.7 0.7 1.0"/>
+  </material>
+  <material name="blue">
+    <color rgba="0.2 0.5 0.8 1.0"/>
+  </material>
+  <!-- ===================== BASE LINK ===================== -->
   <link name="base_link">
-    <!-- Visual: what you see in RViz and Gazebo -->
-    <visual>
-      <geometry>
-        <cylinder radius="${base_radius}" length="${base_height}"/>
-      </geometry>
-      <material name="dark_grey">
-        <color rgba="0.2 0.2 0.2 1.0"/>
-      </material>
-    </visual>
-    <!-- Collision: simplified shape used by physics engine -->
-    <collision>
-      <geometry>
-        <cylinder radius="${base_radius}" length="${base_height}"/>
-      </geometry>
-    </collision>
-    <!-- Inertial: required for Gazebo to simulate physics -->
-    <!-- Inertia tensor for solid cylinder:
-         Ixx = Iyy = m(3r^2 + h^2)/12
-         Izz = mr^2/2 -->
-    <inertial>
-      <mass value="${base_mass}"/>
-      <inertia
-        ixx="${base_mass * (3*base_radius*base_radius + base_height*base_height) / 12}"
-        iyy="${base_mass * (3*base_radius*base_radius + base_height*base_height) / 12}"
-        izz="${base_mass * base_radius*base_radius / 2}"
-        ixy="0.0" ixz="0.0" iyz="0.0"/>
+    <visual>
+      <geometry>
+        <mesh filename="package://arm_description/meshes/base_link.stl" />
+      </geometry>
+      <material name="dark_grey"/>
+    </visual>
+    <collision>
+      <geometry>
+        <mesh filename="package://arm_description/meshes/base_link.stl" />
+      </geometry>
+    </collision>
+    <inertial>
+      <mass value="0.5"/>
+      <inertia ixx="0.001" iyy="0.001" izz="0.001" ixy="0" ixz="0" iyz="0"/>
+    </inertial>
+  </link>
+  <!-- ===================== JOINT 1 — Waist (Z axis) ===================== -->
+  <joint name="joint_1" type="revolute">
+    <parent link="base_link"/>
+    <child link="link_1"/>
+    <!-- Joint sits on top of base: 40mm up -->
+    <origin xyz="0 0 0.04" rpy="0 0 0"/>
+    <axis xyz="0 0 1"/>
+    <limit lower="-3.14159" upper="3.14159" effort="100" velocity="1.0"/>
+  </joint>
+  <!-- ===================== LINK 1 ===================== -->
+  <link name="link_1">
+    <visual>
+      <geometry>
+        <mesh filename="package://arm_description/meshes/link_1.stl" />
+      </geometry>
+      <material name="light_grey"/>
+    </visual>
+    <collision>
+      <geometry>
+        <mesh filename="package://arm_description/meshes/link_1.stl" />
+      </geometry>
+    </collision>
+    <inertial>
+      <mass value="0.4"/>
+      <inertia ixx="0.001" iyy="0.001" izz="0.001" ixy="0" ixz="0" iyz="0"/>
+    </inertial>
+  </link>
+  <!-- ===================== JOINT 2 — Shoulder (Y axis) ===================== -->
+  <joint name="joint_2" type="revolute">
+    <parent link="link_1"/>
+    <child link="link_2"/>
+    <!-- Joint sits on top of link_1: 80mm up -->
+    <origin xyz="0 0 0.08" rpy="0 0 0"/>
+    <axis xyz="0 1 0"/>
+    <limit lower="-1.5708" upper="1.5708" effort="100" velocity="1.0"/>
+  </joint>
+  <!-- ===================== LINK 2 ===================== -->
+  <link name="link_2">
+    <visual>
+      <geometry>
+        <mesh filename="package://arm_description/meshes/link_2.stl" />
+      </geometry>
+      <material name="dark_grey"/>
+    </visual>
+    <collision>
+      <geometry>
+        <mesh filename="package://arm_description/meshes/link_2.stl" />
+      </geometry>
+    </collision>
+    <inertial>
+      <mass value="0.4"/>
+      <inertia ixx="0.001" iyy="0.001" izz="0.001" ixy="0" ixz="0" iyz="0"/>
+    </inertial>
+  </link>
+  <!-- ===================== JOINT 3 — Elbow (Y axis) ===================== -->
+  <joint name="joint_3" type="revolute">
+    <parent link="link_2"/>
+    <child link="link_3"/>
+    <!-- Joint sits on top of link_2: 120mm up -->
+    <origin xyz="0 0 0.12" rpy="0 0 0"/>
+    <axis xyz="0 1 0"/>
+    <limit lower="-1.5708" upper="1.5708" effort="100" velocity="1.0"/>
+  </joint>
+  <!-- ===================== LINK 3 ===================== -->
+  <link name="link_3">
+    <visual>
+      <geometry>
+        <mesh filename="package://arm_description/meshes/link_3.stl" />
+      </geometry>
+      <material name="light_grey"/>
+    </visual>
+    <collision>
+      <geometry>
+        <mesh filename="package://arm_description/meshes/link_3.stl" />
+      </geometry>
+    </collision>
+    <inertial>
+      <mass value="0.3"/>
+      <inertia ixx="0.001" iyy="0.001" izz="0.001" ixy="0" ixz="0" iyz="0"/>
+    </inertial>
+  </link>
+  <!-- ===================== JOINT 4 — Wrist roll (X axis) ===================== -->
+  <joint name="joint_4" type="revolute">
+    <parent link="link_3"/>
+    <child link="link_4"/>
+    <!-- Joint sits on top of link_3: 100mm up -->
+    <origin xyz="0 0 0.10" rpy="0 0 0"/>
+    <axis xyz="1 0 0"/>
+    <limit lower="-3.14159" upper="3.14159" effort="50" velocity="1.5"/>
+  </joint>
+  <!-- ===================== LINK 4 ===================== -->
+  <link name="link_4">
+    <visual>
+      <geometry>
+        <mesh filename="package://arm_description/meshes/link_4.stl" />
+      </geometry>
+      <material name="blue"/>
+    </visual>
+    <collision>
+      <geometry>
+        <mesh filename="package://arm_description/meshes/link_4.stl" />
+      </geometry>
+    </collision>
+    <inertial>
+      <mass value="0.2"/>
+      <inertia ixx="0.0005" iyy="0.0005" izz="0.0005" ixy="0" ixz="0" iyz="0"/>
+    </inertial>
+  </link>
+  <!-- ===================== JOINT 5 — Wrist pitch (Y axis) ===================== -->
+  <joint name="joint_5" type="revolute">
+    <parent link="link_4"/>
+    <child link="link_5"/>
+    <!-- Joint sits on top of link_4: 40mm up -->
+    <origin xyz="0 0 0.04" rpy="0 0 0"/>
+    <axis xyz="0 1 0"/>
+    <limit lower="-1.5708" upper="1.5708" effort="50" velocity="1.5"/>
+  </joint>
+  <!-- ===================== LINK 5 ===================== -->
+  <link name="link_5">
+    <visual>
+      <geometry>
+        <mesh filename="package://arm_description/meshes/link_5.stl" />
+      </geometry>
+      <material name="dark_grey"/>
+    </visual>
+    <collision>
+      <geometry>
+        <mesh filename="package://arm_description/meshes/link_5.stl" />
+      </geometry>
+    </collision>
+    <inertial>
+      <mass value="0.2"/>
+      <inertia ixx="0.0005" iyy="0.0005" izz="0.0005" ixy="0" ixz="0" iyz="0"/>
+    </inertial>
+  </link>
+  <!-- ===================== JOINT 6 — Tool roll (Z axis) ===================== -->
+  <joint name="joint_6" type="revolute">
+    <parent link="link_5"/>
+    <child link="link_6"/>
+    <!-- Joint sits on top of link_5: 35mm up -->
+    <origin xyz="0 0 0.035" rpy="0 0 0"/>
+    <axis xyz="0 0 1"/>
+    <limit lower="-3.14159" upper="3.14159" effort="30" velocity="2.0"/>
+  </joint>
+  <!-- ===================== LINK 6 ===================== -->
+  <link name="link_6">
+    <visual>
+      <geometry>
+        <mesh filename="package://arm_description/meshes/link_6.stl" />
+      </geometry>
+      <material name="blue"/>
+    </visual>
+    <collision>
+      <geometry>
+        <mesh filename="package://arm_description/meshes/link_6.stl" />
+      </geometry>
+    </collision>
+    <inertial>
+      <mass value="0.1"/>
+      <inertia ixx="0.0001" iyy="0.0001" izz="0.0001" ixy="0" ixz="0" iyz="0"/>
+    </inertial>
+  </link>
+  <!-- ===================== TOOL LINK ===================== -->
+  <joint name="tool_joint" type="fixed">
+    <parent link="link_6"/>
+    <child link="tool_link"/>
+    <origin xyz="0 0 0.015" rpy="0 0 0"/>
+  </joint>
+  <link name="tool_link">
+    <!-- Empty link — end effector attaches here -->
+    <inertial>
+      <mass value="0.01"/>
+      <inertia ixx="0.00001" iyy="0.00001" izz="0.00001" ixy="0" ixz="0" iyz="0"/>
     </inertial>
   </link>
